File: circuit/symphon-E/symphon-E.kicad_pcb (KiCad board)
At the start: 2 copper layers, 14 parts, among them J1 display_headers, J10 Potentiometer, J2 power_in, J3 power_in, J4 RINGER_HEADER, J5 ENCODER_HEADER, J6 KEYPAD_HEADER, J7 MIC_HEADER, J8 9MM_HEADER, J9 AUDIO_HEADER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

Commit message: update pcb
Parts:
- moved J8 0.30 mm to (119.4, 94.0)
Routing:
- net GND: track 127.6 -> 128.6 mm
Other:
- board text added: "1"
- board text added: "12V"
- board text added: "8"
- board text added: "Audio"
- board text added: "SCL"
- board text added: "SDA"
Changed lines of the file:
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@@
     (property "Sheetname" "")
     (attr through_hole)
-    (fp_text reference "J3" (at -3.81 2.61 180) (layer "F.SilkS")
+    (fp_text reference "J3" (at 4.11 1.56 180) (layer "F.SilkS")
       (effects (font (size 1 1) (thickness 0.15)))
     )
@@
     (property "Sheetname" "")
     (attr through_hole)
-    (fp_text reference "J6" (at 8.75 3.81 90) (layer "F.SilkS")
+    (fp_text reference "J6" (at -1.61 1.56 90) (layer "F.SilkS")
       (effects (font (size 1 1) (thickness 0.15)))
     )
@@
     (property "Sheetname" "")
     (attr through_hole)
-    (fp_text reference "J4" (at 6.35 2.54) (layer "F.SilkS")
+    (fp_text reference "J4" (at 4.11 1.56) (layer "F.SilkS")
       (effects (font (size 1 1) (thickness 0.15)))
     )
@@
   )
   (footprint "Connector_JST:JST_EH_B2B-EH-A_1x02_P2.50mm_Vertical" (layer "F.Cu")
-    (at 119.08 93.98 -90)
+    (at 119.38 93.98 -90)
     (descr "JST EH series connector, B2B-EH-A (http://www.jst-mfg.com/product/pdf/eng/eEH.pdf), generated with kicad-footprint-generator")
     (tags "connector JST EH vertical")
@@
     (property "Sheetname" "")
     (attr through_hole)
-    (fp_text reference "J8" (at 1.25 3.51 90) (layer "F.SilkS")
+    (fp_text reference "J8" (at -1.61 1.56 90) (layer "F.SilkS")
       (effects (font (size 1 1) (thickness 0.15)))
     )
@@
     (property "Sheetname" "")
     (attr through_hole)
-    (fp_text reference "J1" (at 3.75 3.81 90) (layer "F.SilkS")
+    (fp_text reference "J1" (at -1.61 1.56 90) (layer "F.SilkS")
       (effects (font (size 1 1) (thickness 0.15)))
     )
@@
     (effects (font (size 1 1) (thickness 0.15)))
   )
+  (gr_text "GND\n" (at 83.82 66.04) (layer "F.SilkS")
+    (effects (font (size 1 1) (thickness 0.15)) (justify left))
+  )
   (gr_text "NMOS" (at 93.98 101.6 90) (layer "F.SilkS")
     (effects (font (size 1 1) (thickness 0.15)))
@@
     (effects (font (size 1.5 1.5) (thickness 0.3)))
   )
+  (gr_text "1" (at 115.57 67.31) (layer "F.SilkS")
+    (effects (font (size 1 1) (thickness 0.15)) (justify left))
+  )
   (gr_text "V1.0.0" (at 125.73 49.53 90) (layer "F.SilkS")
     (effects (font (size 1 1) (thickness 0.15)))
@@
     (effects (font (size 1 1) (thickness 0.15)))
   )
+  (gr_text "GND\n" (at 83.82 55.88) (layer "F.SilkS")
+    (effects (font (size 1 1) (thickness 0.15)) (justify left))
+  )
+  (gr_text "SCL\n" (at 115.57 78.74) (layer "F.SilkS")
+    (effects (font (size 1 1) (thickness 0.15)))
+  )
   (gr_text "Synthpone-E" (at 124.46 66.04 90) (layer "F.SilkS")
     (effects (font (size 2 2) (thickness 0.3)))
   )
+  (gr_text "12V" (at 111.76 101.6) (layer "F.SilkS")
+    (effects (font (size 1 1) (thickness 0.15)) (justify left))
+  )
+  (gr_text "5V\n" (at 115.57 81.28) (layer "F.SilkS")
+    (effects (font (size 1 1) (thickness 0.15)))
+  )
+  (gr_text "GND\n" (at 115.57 83.82) (layer "F.SilkS")
+    (effects (font (size 1 1) (thickness 0.15)))
+  )
   (gr_text "ENCODER\n" (at 77.47 87.63 90) (layer "F.SilkS")
     (effects (font (size 1 1) (thickness 0.15)))
@@
     (effects (font (size 1 1) (thickness 0.15)) (justify left))
   )
+  (gr_text "GND\n" (at 121.92 101.6) (layer "F.SilkS")
+    (effects (font (size 1 1) (thickness 0.15)))
+  )
   (gr_text "5V\n" (at 83.82 105.41 90) (layer "F.SilkS")
     (effects (font (size 1 1) (thickness 0.15)) (justify left))
@@
     (effects (font (size 1 1) (thickness 0.15)))
   )
+  (gr_text "GND\n" (at 113.03 93.98) (layer "F.SilkS")
+    (effects (font (size 1 1) (thickness 0.15)) (justify left))
+  )
   (gr_text "A\n" (at 83.82 86.36) (layer "F.SilkS")
     (effects (font (size 1 1) (thickness 0.15)) (justify left))
   )
+  (gr_text "GND\n" (at 109.22 101.6) (layer "F.SilkS")
+    (effects (font (size 1 1) (thickness 0.15)))
+  )
+  (gr_text "Audio\n" (at 111.76 96.52) (layer "F.SilkS")
+    (effects (font (size 1 1) (thickness 0.15)) (justify left))
+  )
+  (gr_text "GND\n" (at 83.82 76.2) (layer "F.SilkS")
+    (effects (font (size 1 1) (thickness 0.15)) (justify left))
+  )
   (gr_text "Ringer" (at 120.65 107.95) (layer "F.SilkS")
     (effects (font (size 1 1) (thickness 0.15)))
   )
+  (gr_text "SDA\n" (at 115.57 76.2) (layer "F.SilkS")
+    (effects (font (size 1 1) (thickness 0.15)))
+  )
   (gr_text "5V\n" (at 83.82 91.44) (layer "F.SilkS")
     (effects (font (size 1 1) (thickness 0.15)) (justify left))
@@
     (effects (font (size 1 1) (thickness 0.15)))
   )
+  (gr_text "8" (at 115.57 49.53) (layer "F.SilkS")
+    (effects (font (size 1 1) (thickness 0.15)) (justify left))
+  )
+  (segment (start 114.3 101.6) (end 118.11 105.41) (width 0.25) (layer "B.Cu") (net 2))
   (segment (start 88.9 101.6) (end 114.3 101.6) (width 0.25) (layer "B.Cu") (net 2))
-  (segment (start 114.3 101.6) (end 118.11 105.41) (width 0.25) (layer "B.Cu") (net 2))
   (segment (start 88.9 104.14) (end 90.225 105.465) (width 0.25) (layer "B.Cu") (net 3))
   (segment (start 110.395 105.465) (end 111.72 104.14) (width 0.25) (layer "B.Cu") (net 3))
   (segment (start 90.225 105.465) (end 110.395 105.465) (width 0.25) (layer "B.Cu") (net 3))
   (segment (start 121.88 104.14) (end 121.88 96.78) (width 0.25) (layer "F.Cu") (net 4))
-  (segment (start 110.545 105.465) (end 120.555 105.465) (width 0.25) (layer "F.Cu") (net 4))
   (segment (start 81.62 66.04) (end 80.295 64.715) (width 0.25) (layer "F.Cu") (net 4))
   (segment (start 83.055 104.905) (end 82.685 105.275) (width 0.25) (layer "F.Cu") (net 4))
@@
   (segment (start 79.955 104.586701) (end 79.955 102.925) (width 0.25) (layer "F.Cu") (net 4))
   (segment (start 81.28 101.6) (end 81.28 93.82) (width 0.25) (layer "F.Cu") (net 4))
+  (segment (start 111.76 106.68) (end 119.34 106.68) (width 0.25) (layer "F.Cu") (net 4))
   (segment (start 81.28 93.82) (end 79.98 92.52) (width 0.25) (layer "F.Cu") (net 4))
   (segment (start 80.295 67.365) (end 81.62 66.04) (width 0.25) (layer "F.Cu") (net 4))
@@
   (segment (start 119.38 83.82) (end 113.03 83.82) (width 0.25) (layer "F.Cu") (net 4))
   (segment (start 79.98 92.52) (end 79.98 77.8) (width 0.25) (layer "F.Cu") (net 4))
-  (segment (start 109.22 104.14) (end 110.545 105.465) (width 0.25) (layer "F.Cu") (net 4))
   (segment (start 113.03 83.82) (end 109.22 80.01) (width 0.25) (layer "F.Cu") (net 4))
   (segment (start 83.055 96.015) (end 83.055 104.905) (width 0.25) (layer "F.Cu") (net 4))
+  (segment (start 109.22 104.14) (end 111.76 106.68) (width 0.25) (layer "F.Cu") (net 4))
   (segment (start 80.295 74.835) (end 80.295 67.365) (width 0.25) (layer "F.Cu") (net 4))
   (segment (start 121.88 96.78) (end 119.08 93.98) (width 0.25) (layer "F.Cu") (net 4))
+  (segment (start 119.34 106.68) (end 121.88 104.14) (width 0.25) (layer "F.Cu") (net 4))
   (segment (start 79.955 102.925) (end 81.28 101.6) (width 0.25) (layer "F.Cu") (net 4))
-  (segment (start 120.555 105.465) (end 121.88 104.14) (width 0.25) (layer "F.Cu") (net 4))
   (segment (start 119.38 93.68) (end 119.38 83.82) (width 0.25) (layer "F.Cu") (net 4))
   (segment (start 82.685 105.275) (end 80.643299 105.275) (width 0.25) (layer "F.Cu") (net 4))
