File: circuit/symphon-E/_autosave-symphon-E.kicad_pcb (KiCad board)
At the start: 2 copper layers, 50.8 x 63.5 mm, 15 parts, among them J1 display_headers, J10 Potentiometer, J2 power_in, J3 power_in, J4 RINGER_HEADER, J5 ENCODER_HEADER, J6 KEYPAD_HEADER, J7 MIC_HEADER, J8 9MM_HEADER, J9 AUDIO_HEADER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

Commit message: update schematic
Routing:
- net AUDIO_OUT: track 85.2 -> 86.8 mm
Changed lines of the file:
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@@
   (segment (start 93.98 67.31) (end 93.98 68.4353) (width 0.25) (layer "F.Cu") (net 10))
   (segment (start 88.9 68.8247) (end 87.8747 67.7994) (width 0.25) (layer "F.Cu") (net 11))
-  (segment (start 87.8747 67.7994) (end 87.8747 57.3947) (width 0.25) (layer "F.Cu") (net 11))
+  (segment (start 86.36 55.88) (end 81.28 50.8) (width 0.25) (layer "F.Cu") (net 11))
+  (segment (start 87.8747 59.9347) (end 86.36 58.42) (width 0.25) (layer "F.Cu") (net 11))
+  (segment (start 86.36 58.42) (end 86.36 55.88) (width 0.25) (layer "F.Cu") (net 11))
   (segment (start 88.9 69.85) (end 88.9 68.8247) (width 0.25) (layer "F.Cu") (net 11))
-  (segment (start 87.8747 57.3947) (end 81.28 50.8) (width 0.25) (layer "F.Cu") (net 11))
+  (segment (start 87.8747 67.7994) (end 87.8747 59.9347) (width 0.25) (layer "F.Cu") (net 11))
   (segment (start 84.0647 73.66) (end 87.8747 69.85) (width 0.25) (layer "B.Cu") (net 11))
   (segment (start 81.62 73.66) (end 84.0647 73.66) (width 0.25) (layer "B.Cu") (net 11))
   (segment (start 88.9 69.85) (end 87.8747 69.85) (width 0.25) (layer "B.Cu") (net 11))
   (segment (start 88.9 70.8845) (end 88.9 77.47) (width 0.25) (layer "F.Cu") (net 12))
+  (segment (start 92.4043 68.8857) (end 90.17 71.12) (width 0.25) (layer "F.Cu") (net 12))
+  (segment (start 110.3453 66.1154) (end 93.5359 66.1154) (width 0.25) (layer "F.Cu") (net 12))
   (segment (start 110.3453 66.1154) (end 110.3453 59.1192) (width 0.25) (layer "F.Cu") (net 12))
-  (segment (start 88.4749 70.8845) (end 81.62 64.0296) (width 0.25) (layer "F.Cu") (net 12))
-  (segment (start 81.62 64.0296) (end 81.62 63.54) (width 0.25) (layer "F.Cu") (net 12))
-  (segment (start 89.3382 70.8845) (end 88.9 70.8845) (width 0.25) (layer "F.Cu") (net 12))
+  (segment (start 92.4043 67.247) (end 92.4043 68.8857) (width 0.25) (layer "F.Cu") (net 12))
   (segment (start 118.4985 95.3047) (end 110.3453 87.1515) (width 0.25) (layer "F.Cu") (net 12))
-  (segment (start 93.5359 66.1154) (end 92.4043 67.247) (width 0.25) (layer "F.Cu") (net 12))
-  (segment (start 92.4043 67.8184) (end 89.3382 70.8845) (width 0.25) (layer "F.Cu") (net 12))
+  (segment (start 88.6645 71.12) (end 87.5352 71.12) (width 0.25) (layer "F.Cu") (net 12))
+  (segment (start 90.17 71.12) (end 88.9 71.12) (width 0.25) (layer "F.Cu") (net 12))
+  (segment (start 87.5352 69.4552) (end 81.62 63.54) (width 0.25) (layer "F.Cu") (net 12))
   (segment (start 119.38 95.3047) (end 118.4985 95.3047) (width 0.25) (layer "F.Cu") (net 12))
   (segment (start 109.5014 58.2753) (end 109.22 58.2753) (width 0.25) (layer "F.Cu") (net 12))
   (segment (start 110.3453 59.1192) (end 109.5014 58.2753) (width 0.25) (layer "F.Cu") (net 12))
+  (segment (start 87.5352 71.12) (end 87.5352 69.4552) (width 0.25) (layer "F.Cu") (net 12))
   (segment (start 110.3453 87.1515) (end 110.3453 66.1154) (width 0.25) (layer "F.Cu") (net 12))
-  (segment (start 110.3453 66.1154) (end 93.5359 66.1154) (width 0.25) (layer "F.Cu") (net 12))
+  (segment (start 93.5359 66.1154) (end 92.4043 67.247) (width 0.25) (layer "F.Cu") (net 12))
   (segment (start 119.38 96.48) (end 119.38 95.3047) (width 0.25) (layer "F.Cu") (net 12))
-  (segment (start 92.4043 67.247) (end 92.4043 67.8184) (width 0.25) (layer "F.Cu") (net 12))
+  (segment (start 88.9 70.8845) (end 88.6645 71.12) (width 0.25) (layer "F.Cu") (net 12))
   (segment (start 109.22 57.15) (end 109.22 58.2753) (width 0.25) (layer "F.Cu") (net 12))
-  (segment (start 88.9 70.8845) (end 88.4749 70.8845) (width 0.25) (layer "F.Cu") (net 12))
   (segment (start 116.98 52.07) (end 119.38 49.67) (width 0.25) (layer "B.Cu") (net 13))
   (segment (start 109.22 52.07) (end 116.98 52.07) (width 0.25) (layer "B.Cu") (net 13))
